File: 2023-2024_senior_design/PCB Design/V0.4.0/CAPSTONE_sensor_unitV0_4.kicad_sch (KiCad schematic)
At the start: 4 parts, among them U1 Teensy4.0-teensy-ARTS-Lab, U2 nRF24L01+-ARTS-Lab

Commit message: PCB Design V0.4.0
Parts:
- A1: footprint Stuff:MPU6050_Module -> Stuff:MPU6050_Sensor_package_edit
- Micro_SD1: footprint Arts:small_microSD_v2 -> Arts:small_microSD_sensor_package_edit
- U1: footprint Arts:Teensy40 -> Arts:Teensy40_sensor_package_edit
- U2: footprint Arts:nRF24L01+ -> Arts:nRF24L01+_sensor_package_edit_V0_2
Connections:
- net at Micro_SD1.1 (3.3V), U2.1 (3.3V): now also U1.31 (3V3); no longer U1.16 (3V3)
- net GND: now reaches Micro_SD1.6 (GND), U1.1 (GND)
- net GND: now also A1.2 (GND), U1.32 (GND), U2.5 (GND)
- net at A1.1 (VCC): now also U1.33 (VIN); no longer U1.34 (VUSB)
- now unconnected: U1.47 (GND)
Changed lines of the file:
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@@
 (kicad_sch (version 20230121) (generator eeschema)
   (paper "A4")
-  (junction (at 60.96 128.27) (diameter 0) (color 0 0 0 0)
+  (junction (at 149.86 123.19) (diameter 0) (color 0 0 0 0)
   )
   (junction (at 60.96 133.35) (diameter 0) (color 0 0 0 0)
@@
   (junction (at 53.34 138.43) (diameter 0) (color 0 0 0 0)
   )
+  (junction (at 48.26 140.97) (diameter 0) (color 0 0 0 0)
+  )
+  (junction (at 180.34 106.68) (diameter 0) (color 0 0 0 0)
+  )
   (junction (at 57.15 135.89) (diameter 0) (color 0 0 0 0)
   )
@@
     (stroke (width 0) (type default))
   )
+  (wire (pts (xy 184.15 110.49) (xy 184.15 106.68))
+    (stroke (width 0) (type default))
+  )
   (wire (pts (xy 58.42 133.35) (xy 60.96 133.35))
     (stroke (width 0) (type default))
@@
     (stroke (width 0) (type default))
   )
-  (wire (pts (xy 59.69 128.27) (xy 60.96 128.27))
-    (stroke (width 0) (type default))
-  )
   (wire (pts (xy 60.96 171.45) (xy 60.96 133.35))
     (stroke (width 0) (type default))
@@
     (stroke (width 0) (type default))
   )
-  (wire (pts (xy 133.35 151.13) (xy 133.35 120.65))
-    (stroke (width 0) (type default))
-  )
-  (wire (pts (xy 53.34 158.75) (xy 53.34 138.43))
+  (wire (pts (xy 180.34 99.06) (xy 180.34 106.68))
     (stroke (width 0) (type default))
   )
@@
     (stroke (width 0) (type default))
   )
-  (wire (pts (xy 149.86 93.98) (xy 154.94 93.98))
-    (stroke (width 0) (type default))
-  )
   (wire (pts (xy 52.07 130.81) (xy 62.23 130.81))
     (stroke (width 0) (type default))
@@
     (stroke (width 0) (type default))
   )
+  (wire (pts (xy 109.22 113.03) (xy 109.22 151.13))
+    (stroke (width 0) (type default))
+  )
   (wire (pts (xy 46.99 38.1) (xy 46.99 140.97))
     (stroke (width 0) (type default))
   )
+  (wire (pts (xy 59.69 128.27) (xy 59.69 123.19))
+    (stroke (width 0) (type default))
+  )
   (wire (pts (xy 83.82 63.5) (xy 93.98 63.5))
     (stroke (width 0) (type default))
@@
     (stroke (width 0) (type default))
   )
-  (wire (pts (xy 149.86 55.88) (xy 180.34 55.88))
-    (stroke (width 0) (type default))
-  )
   (wire (pts (xy 137.16 138.43) (xy 137.16 116.84))
     (stroke (width 0) (type default))
@@
     (stroke (width 0) (type default))
   )
+  (wire (pts (xy 53.34 138.43) (xy 53.34 158.75))
+    (stroke (width 0) (type default))
+  )
+  (wire (pts (xy 48.26 140.97) (xy 48.26 149.86))
+    (stroke (width 0) (type default))
+  )
   (wire (pts (xy 93.98 66.04) (xy 39.37 66.04))
     (stroke (width 0) (type default))
@@
     (stroke (width 0) (type default))
   )
+  (wire (pts (xy 149.86 99.06) (xy 180.34 99.06))
+    (stroke (width 0) (type default))
+  )
   (wire (pts (xy 93.98 43.18) (xy 52.07 43.18))
     (stroke (width 0) (type default))
   )
-  (wire (pts (xy 60.96 128.27) (xy 62.23 128.27))
-    (stroke (width 0) (type default))
-  )
-  (wire (pts (xy 133.35 120.65) (xy 60.96 120.65))
-    (stroke (width 0) (type default))
-  )
-  (wire (pts (xy 154.94 147.32) (xy 180.34 147.32))
+  (wire (pts (xy 156.21 101.6) (xy 156.21 123.19))
+    (stroke (width 0) (type default))
+  )
+  (wire (pts (xy 149.86 101.6) (xy 156.21 101.6))
+    (stroke (width 0) (type default))
+  )
+  (wire (pts (xy 161.29 96.52) (xy 161.29 147.32))
+    (stroke (width 0) (type default))
+  )
+  (wire (pts (xy 46.99 140.97) (xy 48.26 140.97))
+    (stroke (width 0) (type default))
+  )
+  (wire (pts (xy 48.26 140.97) (xy 62.23 140.97))
+    (stroke (width 0) (type default))
+  )
+  (wire (pts (xy 184.15 106.68) (xy 180.34 106.68))
+    (stroke (width 0) (type default))
+  )
+  (wire (pts (xy 180.34 106.68) (xy 180.34 113.03))
     (stroke (width 0) (type default))
   )
@@
     (stroke (width 0) (type default))
   )
+  (wire (pts (xy 156.21 123.19) (xy 149.86 123.19))
+    (stroke (width 0) (type default))
+  )
+  (wire (pts (xy 149.86 96.52) (xy 161.29 96.52))
+    (stroke (width 0) (type default))
+  )
+  (wire (pts (xy 161.29 147.32) (xy 180.34 147.32))
+    (stroke (width 0) (type default))
+  )
   (wire (pts (xy 93.98 38.1) (xy 46.99 38.1))
     (stroke (width 0) (type default))
   )
-  (wire (pts (xy 46.99 140.97) (xy 62.23 140.97))
-    (stroke (width 0) (type default))
-  )
   (wire (pts (xy 93.98 99.06) (xy 87.63 99.06))
     (stroke (width 0) (type default))
   )
-  (wire (pts (xy 60.96 120.65) (xy 60.96 128.27))
-    (stroke (width 0) (type default))
-  )
-  (wire (pts (xy 93.98 76.2) (xy 59.69 76.2))
-    (stroke (width 0) (type default))
-  )
-  (wire (pts (xy 109.22 151.13) (xy 109.22 113.03))
+  (wire (pts (xy 59.69 123.19) (xy 149.86 123.19))
     (stroke (width 0) (type default))
   )
@@
     (stroke (width 0) (type default))
   )
+  (wire (pts (xy 133.35 151.13) (xy 149.86 151.13))
+    (stroke (width 0) (type default))
+  )
   (wire (pts (xy 137.16 116.84) (xy 85.09 116.84))
     (stroke (width 0) (type default))
   )
+  (wire (pts (xy 62.23 128.27) (xy 59.69 128.27))
+    (stroke (width 0) (type default))
+  )
   (wire (pts (xy 143.51 173.99) (xy 143.51 153.67))
     (stroke (width 0) (type default))
   )
-  (wire (pts (xy 154.94 93.98) (xy 154.94 147.32))
-    (stroke (width 0) (type default))
-  )
-  (wire (pts (xy 59.69 76.2) (xy 59.69 128.27))
+  (wire (pts (xy 149.86 123.19) (xy 149.86 151.13))
     (stroke (width 0) (type default))
   )
@@
   )
   (wire (pts (xy 109.22 113.03) (xy 180.34 113.03))
-    (stroke (width 0) (type default))
-  )
-  (wire (pts (xy 180.34 55.88) (xy 180.34 113.03))
     (stroke (width 0) (type default))
   )
@@
       (effects (font (size 1.27 1.27)) (justify left))
     )
-    (property "Footprint" "Arts:small_microSD_v2" (at 82.55 134.62 0)
+    (property "Footprint" "Arts:small_microSD_sensor_package_edit" (at 82.55 134.62 0)
       (effects (font (size 1.27 1.27)) hide)
     )
@@
     (pin "4")
     (instances
-      (project "CAPSTONE_sensor_unit.kicad2_pro"
+      (project "CAPSTONE_sensor_unitV0_4"
         (path "/89cc5cd6-a433-465c-bb2b-4720fbe68ab2"
           (reference "Micro_SD1") (unit 1)
@@
       (effects (font (size 1.27 1.27)) (justify right))
     )
-    (property "Footprint" "Stuff:MPU6050_Module" (at 204.47 143.51 0)
+    (property "Footprint" "Stuff:MPU6050_Sensor_package_edit" (at 204.47 143.51 0)
       (effects (font (size 1.27 1.27)) hide)
     )
@@
     (pin "3")
     (instances
-      (project "CAPSTONE_sensor_unit.kicad2_pro"
+      (project "CAPSTONE_sensor_unitV0_4"
         (path "/89cc5cd6-a433-465c-bb2b-4720fbe68ab2"
           (reference "A1") (unit 1)
+        )
+      )
+    )
+  )
+  (symbol (lib_id "power:GND") (at 184.15 110.49 0) (unit 1)
+    (in_bom yes) (on_board yes) (dnp no) (fields_autoplaced)
+    (property "Reference" "#PWR02" (at 184.15 116.84 0)
+      (effects (font (size 1.27 1.27)) hide)
+    )
+    (property "Value" "GND" (at 184.15 115.57 0)
+      (effects (font (size 1.27 1.27)))
+    )
+    (property "Footprint" "" (at 184.15 110.49 0)
+      (effects (font (size 1.27 1.27)) hide)
+    )
+    (property "Datasheet" "" (at 184.15 110.49 0)
+      (effects (font (size 1.27 1.27)) hide)
+    )
+    (pin "1")
+    (instances
+      (project "CAPSTONE_sensor_unitV0_4"
+        (path "/89cc5cd6-a433-465c-bb2b-4720fbe68ab2"
+          (reference "#PWR02") (unit 1)
         )
       )
@@
       (effects (font (size 1.1938 1.1938)))
     )
-    (property "Footprint" "Arts:nRF24L01+" (at 130.81 153.67 0)
+    (property "Footprint" "Arts:nRF24L01+_sensor_package_edit_V0_2" (at 130.81 153.67 0)
       (effects (font (size 1.27 1.27)) hide)
     )
@@
     (pin "8")
     (instances
-      (project "CAPSTONE_sensor_unit.kicad2_pro"
+      (project "CAPSTONE_sensor_unitV0_4"
         (path "/89cc5cd6-a433-465c-bb2b-4720fbe68ab2"
           (reference "U2") (unit 1)
+        )
+      )
+    )
+  )
+  (symbol (lib_id "power:GND") (at 48.26 149.86 0) (unit 1)
+    (in_bom yes) (on_board yes) (dnp no) (fields_autoplaced)
+    (property "Reference" "#PWR01" (at 48.26 156.21 0)
+      (effects (font (size 1.27 1.27)) hide)
+    )
+    (property "Value" "GND" (at 48.26 154.94 0)
+      (effects (font (size 1.27 1.27)))
+    )
+    (property "Footprint" "" (at 48.26 149.86 0)
+      (effects (font (size 1.27 1.27)) hide)
+    )
+    (property "Datasheet" "" (at 48.26 149.86 0)
+      (effects (font (size 1.27 1.27)) hide)
+    )
+    (pin "1")
+    (instances
+      (project "CAPSTONE_sensor_unitV0_4"
+        (path "/89cc5cd6-a433-465c-bb2b-4720fbe68ab2"
+          (reference "#PWR01") (unit 1)
         )
       )
@@
       (effects (font (size 1.27 1.27)))
     )
-    (property "Footprint" "Arts:Teensy40" (at 111.76 67.31 0)
+    (property "Footprint" "Arts:Teensy40_sensor_package_edit" (at 111.76 67.31 0)
       (effects (font (size 1.27 1.27)) hide)
     )
@@
     (pin "41")
     (instances
-      (project "CAPSTONE_sensor_unit.kicad2_pro"
+      (project "CAPSTONE_sensor_unitV0_4"
         (path "/89cc5cd6-a433-465c-bb2b-4720fbe68ab2"
           (reference "U1") (unit 1)
